File: MahJamma.kicad_pcb (KiCad board)
At the start: 2 copper layers, 118.3 x 38.7 mm, 8 parts, among them J1 JAMMA, J2 UART, J3 BOOT, J4 USB_A, J5 MAHJONG, U1 CH559

Commit message: pcb v1.10
Parts:
- added C3: 0.1u, Capacitor_SMD:C_0603_1608Metric_Pad1.08x0.95mm_HandSolder, F.Cu at (161.3, 68.6)
- added C4: 0.1u, Capacitor_SMD:C_0603_1608Metric_Pad1.08x0.95mm_HandSolder, F.Cu at (148.6, 62.2)
- added C5: 0.1u, Capacitor_SMD:C_0603_1608Metric_Pad1.08x0.95mm_HandSolder, F.Cu at (153.7, 77.5)
- added C6: 0.1u, Capacitor_SMD:C_0603_1608Metric_Pad1.08x0.95mm_HandSolder, F.Cu at (143.5, 69.8)
- added D1: LED, LED_SMD:LED_0603_1608Metric_Pad1.05x0.95mm_HandSolder, F.Cu at (111.8, 77.5)
- added G1: LOGO, toyoshim:mahjamma, F.Cu at (196.8, 62.2)
- added J6: JTAG, Connector_PinHeader_2.54mm:PinHeader_2x05_P2.54mm_Vertical, F.Cu at (185.4, 73.7)
- added R1: 1K, Resistor_SMD:R_0603_1608Metric_Pad0.98x0.95mm_HandSolder, F.Cu at (108.0, 77.5)
- added R2: 10K, Resistor_SMD:R_0603_1608Metric_Pad0.98x0.95mm_HandSolder, F.Cu at (182.9, 69.8)
- added R3: 10K, Resistor_SMD:R_0603_1608Metric_Pad0.98x0.95mm_HandSolder, F.Cu at (180.3, 69.8)
- added R4: 10K, Resistor_SMD:R_0603_1608Metric_Pad0.98x0.95mm_HandSolder, F.Cu at (185.4, 69.8)
- added R5: 10K, Resistor_SMD:R_0603_1608Metric_Pad0.98x0.95mm_HandSolder, F.Cu at (175.3, 69.8)
- added U2: EPM3032A(TQFP), Package_QFP:TQFP-44_10x10mm_P0.8mm, F.Cu at (152.4, 69.8)
- moved J1 2.54 mm to (154.9, 86.4)
- moved C1 1.68 mm to (119.4, 63.1)
- moved C2 1.68 mm to (116.8, 63.1)
- moved J4 0.78 mm to (105.4, 67.3)
Connections:
- net /3.3V renamed +3.3V
- U1 pad 10: /M3 -> unconnected-(U1-Pad10)
- U1 pad 11: /M1 -> unconnected-(U1-Pad11)
- U1 pad 12: /SVC -> unconnected-(U1-Pad12)
- U1 pad 13: /M11 -> unconnected-(U1-Pad13)
- U1 pad 19: unconnected-(U1-Pad19) -> /COIN
- U1 pad 20: unconnected-(U1-Pad20) -> /SVC
- U1 pad 21: unconnected-(U1-Pad21) -> /LED
- U1 pad 22: unconnected-(U1-Pad22) -> /S_RON
- U1 pad 23: unconnected-(U1-Pad23) -> /S_REACH
- U1 pad 24: unconnected-(U1-Pad24) -> /S_KAN
- U1 pad 25: unconnected-(U1-Pad25) -> /S_PON
- U1 pad 26: unconnected-(U1-Pad26) -> /S_CHI
- U1 pad 27: unconnected-(U1-Pad27) -> /S_N
- U1 pad 28: unconnected-(U1-Pad28) -> /S_M
- U1 pad 33: /M6 -> /S_L
- U1 pad 34: /M10 -> /S_K
- U1 pad 35: /M9 -> /S_J
- U1 pad 36: /M2 -> /S_I
- U1 pad 38: unconnected-(U1-Pad38) -> /S_H
- U1 pad 39: unconnected-(U1-Pad39) -> /S_G
- U1 pad 40: unconnected-(U1-Pad40) -> /S_F
- U1 pad 43: unconnected-(U1-Pad43) -> /S_E
- U1 pad 44: unconnected-(U1-Pad44) -> /S_D
- U1 pad 45: unconnected-(U1-Pad45) -> /S_C
- U1 pad 46: unconnected-(U1-Pad46) -> /S_B
- U1 pad 47: unconnected-(U1-Pad47) -> /S_A
- U1 pad 48: unconnected-(U1-Pad48) -> /S_START
- U1 pad 7: /M8 -> unconnected-(U1-Pad7)
- U1 pad 8: /M7 -> unconnected-(U1-Pad8)
- U1 pad 9: /M4 -> unconnected-(U1-Pad9)
Routing:
- net +3.3V: track 2.96 -> 69.5 mm, vias 0 -> 6
- net /M9: track 32.4 -> 91.3 mm
- net /M2: track 27.5 -> 82.4 mm, vias 2 -> 4
- net VCC: track 227.3 -> 280.6 mm, vias 17 -> 21
- net /S_START: track 0.00 -> 49.3 mm, vias 0 -> 2
- net /S_D: track 0.00 -> 47.8 mm, vias 0 -> 4
- net /S_B: track 0.00 -> 47.7 mm, vias 0 -> 4
- net /M10: track 33.9 -> 80.2 mm, vias 2 -> 0
- net /TCK: track 0.00 -> 45.8 mm, vias 0 -> 2
- net /S_A: track 0.00 -> 45.3 mm, vias 0 -> 4
- net /M1: track 59.5 -> 16.4 mm, vias 3 -> 1
- net /S_C: track 0.00 -> 41.4 mm, vias 0 -> 4
- net /TMS: track 0.00 -> 41.4 mm, vias 0 -> 2
- net /S_RON: track 0.00 -> 40.5 mm
- net /M3: track 55.6 -> 18.4 mm, vias 3 -> 1
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Other:
- board size 118.3 x 38.7 mm -> 118.3 x 41.3 mm
- board text added: "Ver 1.10 2022.10.11 Designed by Mellow PCB"
- board text removed: "Ver 1.00 2022.08.27 Designed by Mellow PCB"

Commit message: v1.20
Parts:
- removed R2, R3, R4, R5: 10K, Resistor_SMD:R_0603_1608Metric_Pad0.98x0.95mm_HandSolder
- moved C5 24.3 mm to (130.6, 69.8), turned to 90 degrees
- moved C3 21.7 mm to (141.1, 76.5)
- moved J2 20.1 mm to (109.2, 77.5)
- moved J3 20.1 mm to (105.4, 77.5)
- moved U2 14.6 mm to (137.8, 69.2), turned to 90 degrees
- moved C6 9.97 mm to (137.9, 61.6), turned to 0 degrees
- moved C4 7.92 mm to (145.7, 69.6), turned to -90 degrees
- moved D1 5.44 mm to (117.2, 77.5)
- moved R1 5.44 mm to (113.4, 77.5)
- moved U1 2.62 mm to (116.8, 69.8)
- moved C1 1.42 mm to (118.0, 62.9)
- moved C2 0.26 mm to (116.7, 62.9)
Connections:
- U1 pad 10: unconnected-(U1-Pad10) -> /M6
- U1 pad 11: unconnected-(U1-Pad11) -> /M2
- U1 pad 12: unconnected-(U1-Pad12) -> /M9
- U1 pad 13: unconnected-(U1-Pad13) -> /M10
- U1 pad 14: unconnected-(U1-Pad14) -> /KEY_2
- U1 pad 15: unconnected-(U1-Pad15) -> /KEY_3
- U1 pad 17: unconnected-(U1-Pad17) -> /KEY_4
- U1 pad 19: /COIN -> /KEY_5
- U1 pad 20: /SVC -> /KEY_6
- U1 pad 21: /LED -> /KEY_7
- U1 pad 22: /S_RON -> /KEY_8
- U1 pad 23: /S_REACH -> /KEY_9
- U1 pad 24: /S_KAN -> /KEY_10
- U1 pad 25: /S_PON -> /KEY_11
- U1 pad 26: /S_CHI -> /KEY_12
- U1 pad 27: /S_N -> /KEY_13
- U1 pad 28: /S_M -> /KEY_14
- U1 pad 33: /S_L -> /KEY_CLK_0
- U1 pad 34: /S_K -> /MAT_EN_X_1
- U1 pad 35: /S_J -> /MAT_EN_X_0
- U1 pad 36: /S_I -> /KEY_CLK_1
- U1 pad 38: /S_H -> /MAT_P
- U1 pad 39: /S_G -> unconnected-(U1-Pad39)
- U1 pad 40: /S_F -> /1PC
- U1 pad 43: /S_E -> /M11
- U1 pad 44: /S_D -> /M1
- U1 pad 45: /S_C -> /M3
- U1 pad 46: /S_B -> /M4
- U1 pad 47: /S_A -> /M7
- U1 pad 48: /S_START -> /M8
- U1 pad 5: unconnected-(U1-Pad5) -> /KEY_0
- U1 pad 6: unconnected-(U1-Pad6) -> /KEY_1
- U1 pad 7: unconnected-(U1-Pad7) -> /SVC
- U1 pad 8: unconnected-(U1-Pad8) -> /LED
- U1 pad 9: unconnected-(U1-Pad9) -> /M5
- U2 pad 10: /S_E -> /KEY_4
- U2 pad 12: /S_F -> /KEY_3
- U2 pad 13: /S_G -> /KEY_2
- U2 pad 14: /S_H -> /KEY_1
- U2 pad 15: /S_I -> /KEY_0
- U2 pad 18: /S_J -> /M11
- U2 pad 19: /S_K -> /M1
- U2 pad 2: /S_START -> /KEY_9
- U2 pad 20: /S_L -> /M3
- U2 pad 21: /S_M -> /M4
- U2 pad 22: /S_N -> /M7
- U2 pad 23: /S_CHI -> /M8
- U2 pad 25: /S_PON -> /M2
- U2 pad 27: /S_KAN -> /M6
- U2 pad 28: /S_REACH -> /M10
- U2 pad 3: /S_A -> /KEY_8
- U2 pad 31: /S_RON -> /M9
- U2 pad 33: /M10 -> /KEY_14
- U2 pad 34: /M2 -> /KEY_13
- U2 pad 35: /M9 -> /KEY_12
- U2 pad 37: /M6 -> /KEY_CLK_0
- U2 pad 38: /M11 -> /MAT_EN_X_1
- U2 pad 39: /M8 -> /MAT_EN_X_0
- U2 pad 40: /M7 -> /KEY_CLK_1
- U2 pad 42: /M4 -> /MAT_P
- U2 pad 43: /M3 -> /KEY_11
- U2 pad 44: /M1 -> /KEY_10
- U2 pad 5: /S_B -> /KEY_7
- U2 pad 6: /S_C -> /KEY_6
- U2 pad 8: /S_D -> /KEY_5
Routing:
- net /S_START: track 49.3 -> 0.00 mm, vias 2 -> 0
- net /S_D: track 47.8 -> 0.00 mm, vias 4 -> 0
- net /S_B: track 47.7 -> 0.00 mm, vias 4 -> 0
- net /KEY_2: track 0.00 -> 45.4 mm, vias 0 -> 2
- net /S_A: track 45.3 -> 0.00 mm, vias 4 -> 0
- net /KEY_3: track 0.00 -> 41.4 mm, vias 0 -> 2
- net /S_C: track 41.4 -> 0.00 mm, vias 4 -> 0
- net GND: track 534.6 -> 575.1 mm, vias 22 -> 19
- net /S_RON: track 40.5 -> 0.00 mm
- net /M1: track 16.4 -> 54.6 mm, vias 1 -> 3
- net /S_E: track 35.7 -> 0.00 mm, vias 2 -> 0
- net /S_REACH: track 35.3 -> 0.00 mm
- net /12V: track 41.9 -> 76.6 mm, vias 4 -> 7
- net /M9: track 91.3 -> 57.5 mm
- net /M11: track 26.9 -> 60.7 mm, vias 1 -> 3
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- added copper zone on F.Cu, net +3.3V
Other:
- board text added: "Ver 1.20 2022.11.15 Designed by Mellow PCB"
- board text removed: "Ver 1.10 2022.10.11 Designed by Mellow PCB"
