File: MahJamma.kicad_sch (KiCad schematic)
At the start: 8 parts, among them J1 JAMMA, J2 UART, J3 BOOT, J4 USB_A, J5 MAHJONG, U1 CH559

Commit message: pcb v1.10
Parts:
- added C3, C4, C5, C6: 0.1u, Capacitor_SMD:C_0603_1608Metric_Pad1.08x0.95mm_HandSolder, symbol Device:C
- added D1: LED, LED_SMD:LED_0603_1608Metric_Pad1.05x0.95mm_HandSolder, symbol Device:LED
- added J6: JTAG, Connector_PinHeader_2.54mm:PinHeader_2x05_P2.54mm_Vertical, symbol Connector_Generic:Conn_02x05_Odd_Even
- added R1: 1K, Resistor_SMD:R_0603_1608Metric_Pad0.98x0.95mm_HandSolder, symbol Device:R
- added R2, R3, R4, R5: 10K, Resistor_SMD:R_0603_1608Metric_Pad0.98x0.95mm_HandSolder, symbol Device:R
- added U2: EPM3032A(TQFP), Package_QFP:TQFP-44_10x10mm_P0.8mm, symbol toyoshim:EPM3032A(TQFP)
Connections:
- net GND: now also C3.2, C4.2, C5.2, C6.2, J6.10 (Pin_10), J6.2 (Pin_2), R4.1, U2.11 (GND), U2.16 (GND), U2.24 (GND), U2.30 (GND), U2.36 (GND), U2.4 (GND)
- net M1: now also U2.44 (I/O); no longer U1.11 (P3_5)
- net M10: now also U2.33 (I/O); no longer U1.34 (P0_6)
- net M11: now also U2.38 (INPUT/OE1); no longer U1.13 (P3_7)
- net M2: now also U2.34 (I/O); no longer U1.36 (P0_4)
- net M3: now also U2.43 (I/O); no longer U1.10 (P3_4)
- net M4: now also U2.42 (I/O); no longer U1.9 (P3_3)
- net M6: now also U2.37 (INPUT/GCLK1); no longer U1.33 (P0_7)
- net M7: now also U2.40 (INPUT/OE2/GCLK2); no longer U1.8 (P3_2)
- net M8: now also U2.39 (INPUT/GCLRn); no longer U1.7 (P3_1)
- net M9: now also U2.35 (I/O); no longer U1.35 (P0_5)
- net SVC: now also U1.20 (P4_0); no longer U1.12 (P3_6)
- net VCC: now also J6.4 (Pin_4), R1.1, R2.2, R3.2, R5.2
- net COIN: now reaches U1.19 (P4_1)
- net LED: now reaches U1.21 (P2_0)
- net LED: now also D1.1 (K)
- net S_RON: now reaches U1.22 (P2_1)
- net S_RON: now also U2.31 (I/O)
- net S_REACH: now reaches U1.23 (P2_2)
- net S_REACH: now also U2.28 (I/O)
- net S_KAN: now reaches U1.24 (P2_3)
- net S_KAN: now also U2.27 (I/O)
- net S_PON: now reaches U1.25 (P2_4)
- net S_PON: now also U2.25 (I/O)
- net S_CHI: now reaches U1.26 (P2_5)
- net S_CHI: now also U2.23 (I/O)
- net S_N: now reaches U1.27 (P2_6)
- net S_N: now also U2.22 (I/O)
- net S_M: now reaches U1.28 (P2_7)
- net S_M: now also U2.21 (I/O)
- net S_H: now reaches U1.38 (P0_2)
- net S_H: now also U2.14 (I/O)
- net S_G: now reaches U1.39 (P0_1)
- net S_G: now also U2.13 (I/O)
- net S_F: now reaches U1.40 (P0_0)
- net S_F: now also U2.12 (I/O)
- net S_E: now reaches U1.43 (P1_0)
- net S_E: now also U2.10 (I/O)
- net S_D: now reaches U1.44 (P1_1)
- net S_D: now also U2.8 (I/O)
- net S_C: now reaches U1.45 (P1_2)
- net S_C: now also U2.6 (I/O)
- net S_B: now reaches U1.46 (P1_3)
- net S_B: now also U2.5 (I/O)
- net S_A: now reaches U1.47 (P1_4)
- net S_A: now also U2.3 (I/O)
- net S_START: now reaches U1.48 (P1_5)
- net S_START: now also U2.2 (I/O)
- net 3.3V renamed +3.3V
- net +3.3V: now also C3.1, C4.1, C5.1, C6.1, U2.17 (VCC), U2.29 (VCC), U2.41 (VCC), U2.9 (VCC)
- new net: D1.2 (A), R1.2
- new net S_I: U1.36 (P0_4), U2.15 (I/O)
- new net S_J: U1.35 (P0_5), U2.18 (I/O)
- new net S_K: U1.34 (P0_6), U2.19 (I/O)
- new net S_L: U1.33 (P0_7), U2.20 (I/O)
- new net TCK: J6.1 (Pin_1), R4.2, U2.26 (I/O/TCK)
- new net TDI: J6.9 (Pin_9), R5.1, U2.1 (I/O/TDI)
- new net TDO: J6.3 (Pin_3), R2.1, U2.32 (I/O/TDO)
- new net TMS: J6.5 (Pin_5), R3.1, U2.7 (I/O/TMS)
- no-connect marks 80 -> 71
Other:
- moved on the sheet: C1, C2

Commit message: v1.20
Parts:
- removed R2, R3, R4, R5: 10K, Resistor_SMD:R_0603_1608Metric_Pad0.98x0.95mm_HandSolder, symbol Device:R
Connections:
- net 1PC: now also U1.40 (P0_0)
- net LED: now also U1.8 (P3_2); no longer U1.21 (P2_0)
- net M1: now also U1.44 (P1_1), U2.19 (I/O); no longer U2.44 (I/O)
- net M10: now also U1.13 (P3_7), U2.28 (I/O); no longer U2.33 (I/O)
- net M11: now also U1.43 (P1_0), U2.18 (I/O); no longer U2.38 (INPUT/OE1)
- net M2: now also U1.11 (P3_5), U2.25 (I/O); no longer U2.34 (I/O)
- net M3: now also U1.45 (P1_2), U2.20 (I/O); no longer U2.43 (I/O)
- net M4: now also U1.46 (P1_3), U2.21 (I/O); no longer U2.42 (I/O)
- net M5: now also U1.9 (P3_3)
- net M6: now also U1.10 (P3_4), U2.27 (I/O); no longer U2.37 (INPUT/GCLK1)
- net M7: now also U1.47 (P1_4), U2.22 (I/O); no longer U2.40 (INPUT/OE2/GCLK2)
- net M8: now also U1.48 (P1_5), U2.23 (I/O); no longer U2.39 (INPUT/GCLRn)
- net M9: now also U1.12 (P3_6), U2.31 (I/O); no longer U2.35 (I/O)
- net SVC: now also U1.7 (P3_1); no longer U1.20 (P4_0)
- net KEY_2: now reaches U1.14 (P4_3)
- net KEY_2: now also U2.13 (I/O)
- net KEY_3: now reaches U1.15 (P4_2)
- net KEY_3: now also U2.12 (I/O)
- net KEY_4: now reaches U1.17 (P4_7)
- net KEY_4: now also U2.10 (I/O)
- net KEY_0: now reaches U1.5 (P4_5)
- net KEY_0: now also U2.15 (I/O)
- net KEY_1: now reaches U1.6 (P4_4)
- net KEY_1: now also U2.14 (I/O)
- net COIN renamed KEY_5
- net KEY_5: now also U2.8 (I/O)
- net S_A renamed KEY_8
- net KEY_8: now also U1.22 (P2_1); no longer U1.47 (P1_4)
- net S_B renamed KEY_7
- net KEY_7: now also U1.21 (P2_0); no longer U1.46 (P1_3)
- net S_C renamed KEY_6
- net KEY_6: now also U1.20 (P4_0); no longer U1.45 (P1_2)
- net S_CHI renamed KEY_12
- net KEY_12: now also U2.35 (I/O); no longer U2.23 (I/O)
- removed net S_D: U1.44 (P1_1), U2.8 (I/O)
- removed net S_E: U1.43 (P1_0), U2.10 (I/O)
- removed net S_F: U1.40 (P0_0), U2.12 (I/O)
- net S_G: no longer names the net of U1.39 (P0_1)
- net S_G: no longer U2.13 (I/O)
- net S_H renamed MAT_P
- net MAT_P: now also U2.42 (I/O); no longer U2.14 (I/O)
- net S_I renamed KEY_CLK_1
- net KEY_CLK_1: now also U2.40 (INPUT/OE2/GCLK2); no longer U2.15 (I/O)
- net S_J renamed MAT_EN_X_0
- net MAT_EN_X_0: now also U2.39 (INPUT/GCLRn); no longer U2.18 (I/O)
- net S_K renamed MAT_EN_X_1
- net MAT_EN_X_1: now also U2.38 (INPUT/OE1); no longer U2.19 (I/O)
- net S_KAN renamed KEY_10
- net KEY_10: now also U2.44 (I/O); no longer U2.27 (I/O)
- net S_L renamed KEY_CLK_0
- net KEY_CLK_0: now also U2.37 (INPUT/GCLK1); no longer U2.20 (I/O)
- net S_M renamed KEY_14
- net KEY_14: now also U2.33 (I/O); no longer U2.21 (I/O)
- net S_N renamed KEY_13
- net KEY_13: now also U2.34 (I/O); no longer U2.22 (I/O)
- net S_PON renamed KEY_11
- net KEY_11: now also U2.43 (I/O); no longer U2.25 (I/O)
- net S_REACH renamed KEY_9
- net KEY_9: now also U2.2 (I/O); no longer U2.28 (I/O)
- removed net S_RON: U1.22 (P2_1), U2.31 (I/O)
- removed net S_START: U1.48 (P1_5), U2.2 (I/O)
- no-connect marks 71 -> 60
